File: RavenExpander.kicad_pcb (KiCad board)
At the start: 2 copper layers, 21.8 x 20.8 mm, 3 parts, among them J1 CONN_06SMD_MALE, J2 Screw_Terminal_01x04, J3 Screw_Terminal_01x02

Commit message: Add silkscreen
Other:
- board text added: "Rev 1"
- board text added: "Simpler Circuit"
Changed lines of the file:
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@@
   (general
     (thickness 1.6)
-    (drawings 10)
+    (drawings 12)
     (tracks 7)
     (zones 0)
@@
     )
   )
+  (gr_text "Rev 1" (at 131.064 83.312) (layer B.SilkS)
+    (effects (font (size 1.5 1.5) (thickness 0.3)) (justify mirror))
+  )
+  (gr_text "Simpler\nCircuit" (at 140.716 82.296) (layer B.SilkS)
+    (effects (font (size 1.5 1.5) (thickness 0.3)) (justify mirror))
+  )
   (gr_text Main (at 136.652 80.264 90) (layer F.SilkS)
